File: Hardware/DaisyMultiFX/DaisyMultiFX.kicad_sch (KiCad schematic)
At the start: 0 parts

Commit message: Added hardware and the vscode tasks.
Parts:
- added A1: Electrosmith_Daisy_Seed_Rev4, Module:Electrosmith_Daisy_Seed, symbol MCU_Module:Electrosmith_Daisy_Seed_Rev4
- added J1: DC JACK, Connector_JST:JST_PH_B3B-PH-K_1x03_P2.00mm_Vertical, symbol Connector:Conn_01x03_Socket
- added J2: AUDIO_IN_TRS, Connector_Audio:Jack_6.35mm_Neutrik_NMJ6HCD2_Horizontal, symbol Connector_Audio:NMJ6HCD2
- added J3: AUDIO_OUT_TRS, Connector_Audio:Jack_6.35mm_Neutrik_NMJ6HCD2_Horizontal, symbol Connector_Audio:NMJ6HCD2
- added J4: J_AUDIO_IN, Connector_JST:JST_PH_B3B-PH-K_1x03_P2.00mm_Vertical, symbol Connector:Conn_01x03_Socket
- added J5: J_AUDIO_OUT, Connector_JST:JST_PH_B3B-PH-K_1x03_P2.00mm_Vertical, symbol Connector:Conn_01x03_Socket
Connections:
- new net +3.3V: A1.38 (3V3_D)
- new net +3.3VA: A1.21 (3V3_A)
- new net +9V: A1.39 (VIN)
- new net AUDIO_IN_BUFFER_LEFT: A1.16 (AUDIO_IN_1)
- new net AUDIO_IN_BUFFER_RIGHT: A1.17 (AUDIO_IN_2)
- new net AUDIO_IN_JACK_LEFT: J2.T, J4.1 (Pin_1)
- new net AUDIO_IN_JACK_RIGHT: J2.R, J4.2 (Pin_2)
- new net AUDIO_OUT_BUFFER_LEFT: A1.18 (AUDIO_OUT_1)
- new net AUDIO_OUT_BUFFER_RIGHT: A1.19 (AUDIO_OUT_2)
- new net AUDIO_OUT_JACK_LEFT: J3.T, J5.1 (Pin_1)
- new net AUDIO_OUT_JACK_RIGHT: J3.R, J5.2 (Pin_2)
- new net ENC_1_A: A1.1 (USB_ID)
- new net ENC_1_B: A1.2 (SD_DATA_3)
- new net ENC_2_A: A1.3 (SD_DATA_2)
- new net ENC_2_B: A1.4 (SD_DATA_1)
- new net ENC_3_A: A1.5 (SD_DATA_0)
- new net ENC_3_B: A1.6 (SD_CMD)
- new net ENC_4_A: A1.12 (I2C1_SCL)
- new net ENC_4_B: A1.13 (I2C1_SDA)
- new net ENC_MASTER_A: A1.14 (USART1_TX)
- new net ENC_MASTER_B: A1.15 (USART1_RX)
- new net ENC_MASTER_SW: A1.7 (SD_CLK)
- new net FOOT_SWITCH_1: A1.24 (ADC_2)
- new net FOOT_SWITCH_2: A1.25 (ADC_3)
- new net FOOT_SWITCH_3: A1.26 (ADC_4)
- new net GND: A1.20 (AGND), A1.40 (DGND), J1.2 (Pin_2), J1.3 (Pin_3), J2.RN, J2.S, J2.SN, J2.TN, J3.RN, J3.S, J3.SN, J3.TN, J4.3 (Pin_3), J5.3 (Pin_3)
- new net LCD_BL: A1.36 (USB_D_-)
- new net LCD_CS: A1.8 (SPI1_CS)
- new net LCD_DC: A1.33 (SAI2_SD_A)
- new net LCD_MOSI: A1.11 (SPI1_PICO)
- new net LCD_RST: A1.34 (SAI2_FS)
- new net LCD_SCK: A1.9 (SPI1_SCK)
- new net POWER_JACK_PWR: J1.1 (Pin_1)
- no-connect marks 0 -> 11
Other:
- added sheet Controls (Controls.kicad_sch)
- added sheet InputBuffer (InputBuffer.kicad_sch)
- added sheet OutputBuffer (OutputBuffer.kicad_sch)
- added sheet Power (Power.kicad_sch)
- added sheet Screen (Screen.kicad_sch)
